Commit message: updates.

File: vtol_description/urdf/vtol.urdf (robot description, URDF)
Before this commit: robot vtol, 17 links, 16 joints
Links:
- added link cam_back_link, mass 0.01; visual box size=0.03 0.03 0.03
- added link cam_down_link, mass 0.01; visual box size=0.03 0.03 0.03
- added link cam_front_link, mass 0.01; visual box size=0.03 0.03 0.03
- added link cam_left_link, mass 0.01; visual box size=0.03 0.03 0.03
- added link cam_right_link, mass 0.01; visual box size=0.03 0.03 0.03
- added link cam_up_link, mass 0.01; visual box size=0.03 0.03 0.03
Joints:
- added joint cam_back_joint: type fixed, parent base_link, child cam_back_link, origin xyz=0 0 -0.95 rpy=0 1.5708 1.5708
- added joint cam_down_joint: type fixed, parent base_link, child cam_down_link, origin xyz=0 -0.1 -0.05 rpy=0 0 1.5708
- added joint cam_front_joint: type fixed, parent base_link, child cam_front_link, origin xyz=0 0 0.15 rpy=0 -1.5708 -1.5708
- added joint cam_left_joint: type fixed, parent base_link, child cam_left_link, origin xyz=-0.25 0 -0.05 rpy=1.5708 0 3.14159
- added joint cam_right_joint: type fixed, parent base_link, child cam_right_link, origin xyz=0.25 0 -0.05 rpy=-1.5708 0 0
- added joint cam_up_joint: type fixed, parent base_link, child cam_up_link, origin xyz=0 0.1 -0.05 rpy=3.14159 0 1.5708
